File: RelayBoard/RelayBoard.sch (KiCad schematic (older format))
At the start: 17 parts, among them K1 CONN_3, K2 CONN_3, K3 CONN_3, Q1 2N4401, Q2 2N4401, Q3 2N4401

Commit message: Completed RelayBoard PCB Design
Parts:
- renumbered K2 to K1, K3 to K2, K1 to K3
Changed lines of the file:
@@
 LIBS:myTransistors
 LIBS:Relays
+LIBS:RelayBoard-cache
 EELAYER 27 0
 EELAYER END
@@
 	2200 3450 2300 3450
 $Comp
-L CONN_3 K2
+L CONN_3 K1
 U 1 1 535E3856
 P 3950 1400
-F 0 "K2" V 3900 1400 50  0000 C CNN
+F 0 "K1" V 3900 1400 50  0000 C CNN
 F 1 "CONN_3" V 4000 1400 40  0000 C CNN
 F 2 "" H 3950 1400 60  0000 C CNN
@@
 	3400 1400 3600 1400
 $Comp
-L CONN_3 K3
+L CONN_3 K2
 U 1 1 535E38EC
 P 3950 2450
-F 0 "K3" V 3900 2450 50  0000 C CNN
+F 0 "K2" V 3900 2450 50  0000 C CNN
 F 1 "CONN_3" V 4000 2450 40  0000 C CNN
 F 2 "" H 3950 2450 60  0000 C CNN
@@
 $EndComp
 $Comp
-L CONN_3 K1
+L CONN_3 K3
 U 1 1 535E38F2
 P 3900 3550
-F 0 "K1" V 3850 3550 50  0000 C CNN
+F 0 "K3" V 3850 3550 50  0000 C CNN
 F 1 "CONN_3" V 3950 3550 40  0000 C CNN
 F 2 "" H 3900 3550 60  0000 C CNN
@@
 	3450 3550 3550 3550
 $Comp
-L GND #PWR?
+L GND #PWR01
 U 1 1 5364111C
 P 1350 4150
-F 0 "#PWR?" H 1350 4150 30  0001 C CNN
+F 0 "#PWR01" H 1350 4150 30  0001 C CNN
 F 1 "GND" H 1350 4080 30  0001 C CNN
 F 2 "" H 1350 4150 60  0000 C CNN
@@
 $EndComp
 $Comp
-L GND #PWR?
+L GND #PWR02
 U 1 1 53641175
 P 1800 3850
-F 0 "#PWR?" H 1800 3850 30  0001 C CNN
+F 0 "#PWR02" H 1800 3850 30  0001 C CNN
 F 1 "GND" H 1800 3780 30  0001 C CNN
 F 2 "" H 1800 3850 60  0000 C CNN
@@
 $EndComp
 $Comp
-L GND #PWR?
+L GND #PWR03
 U 1 1 53641193
 P 1800 2700
-F 0 "#PWR?" H 1800 2700 30  0001 C CNN
+F 0 "#PWR03" H 1800 2700 30  0001 C CNN
 F 1 "GND" H 1800 2630 30  0001 C CNN
 F 2 "" H 1800 2700 60  0000 C CNN
@@
 $EndComp
 $Comp
-L GND #PWR?
+L GND #PWR04
 U 1 1 536411A0
 P 1800 1700
-F 0 "#PWR?" H 1800 1700 30  0001 C CNN
+F 0 "#PWR04" H 1800 1700 30  0001 C CNN
 F 1 "GND" H 1800 1630 30  0001 C CNN
 F 2 "" H 1800 1700 60  0000 C CNN
@@
 $EndComp
 $Comp
-L GND #PWR?
+L GND #PWR05
 U 1 1 536411A6
 P 1350 850
-F 0 "#PWR?" H 1350 850 30  0001 C CNN
+F 0 "#PWR05" H 1350 850 30  0001 C CNN
 F 1 "GND" H 1350 780 30  0001 C CNN
 F 2 "" H 1350 850 60  0000 C CNN
@@
 $EndComp
 $Comp
-L VCC #PWR?
+L VCC #PWR06
 U 1 1 536411B5
 P 1150 850
-F 0 "#PWR?" H 1150 950 30  0001 C CNN
+F 0 "#PWR06" H 1150 950 30  0001 C CNN
 F 1 "VCC" H 1150 950 30  0000 C CNN
 F 2 "" H 1150 850 60  0000 C CNN
@@
 $EndComp
 $Comp
-L VCC #PWR?
+L VCC #PWR07
 U 1 1 536411D3
 P 2600 1150
-F 0 "#PWR?" H 2600 1250 30  0001 C CNN
+F 0 "#PWR07" H 2600 1250 30  0001 C CNN
 F 1 "VCC" H 2600 1250 30  0000 C CNN
 F 2 "" H 2600 1150 60  0000 C CNN
@@
 $EndComp
 $Comp
-L VCC #PWR?
+L VCC #PWR08
 U 1 1 536411F6
 P 2600 2150
-F 0 "#PWR?" H 2600 2250 30  0001 C CNN
+F 0 "#PWR08" H 2600 2250 30  0001 C CNN
 F 1 "VCC" H 2600 2250 30  0000 C CNN
 F 2 "" H 2600 2150 60  0000 C CNN
@@
 $EndComp
 $Comp
-L VCC #PWR?
+L VCC #PWR09
 U 1 1 53641205
 P 2650 3250
-F 0 "#PWR?" H 2650 3350 30  0001 C CNN
+F 0 "#PWR09" H 2650 3350 30  0001 C CNN
 F 1 "VCC" H 2650 3350 30  0000 C CNN
 F 2 "" H 2650 3250 60  0000 C CNN
